File: 3872_PCB/ECE3872B_4B_PCB_OChristmasTree_board/project.brd (EAGLE design)
At the start: 76.2 x 88.9 mm, 24 parts, among them IC1 74HC08N, J1 1X2-3.5MM, J2 1X2-3.5MM, J3 1X2-3.5MM, J4 1X2-3.5MM

Commit message: Added annotations to the schematic and added a power connection to the quad AND gate IC and regenerated Gerber/drill files
Connections:
- removed net VCC: IC1.14
- net VIN: now also IC1.14
Changed lines of the file:
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@@
 </polygon>
-</signal>
-<signal name="VCC">
-<contactref element="IC1" pad="14"/>
 </signal>
 <signal name="D13">
@@
 <wire x1="42.23" y1="12.7" x2="39.878" y2="12.7" width="0.3048" layer="1"/>
 <via x="39.878" y="12.7" extent="1-16" drill="0.6"/>
+<contactref element="IC1" pad="14"/>
 </signal>
 <signal name="A7">
