File: 3872_PCB/ECE3872B_4B_PCB_OChristmasTree_board/project.sch (EAGLE design)
At the start: 24 parts, among them IC1 74HC08N, J1 1X2-3.5MM, J2 1X2-3.5MM, J3 1X2-3.5MM, J4 1X2-3.5MM

Commit message: Added annotations to the schematic and added a power connection to the quad AND gate IC and regenerated Gerber/drill files
Connections:
- net VIN: now also IC1P.VCC
Other:
- note added: "Both servos use the same power terminal block"
- note added: "Female header pins for Arduino Nano. The microcontroller will get power from the 5V into the board"
- note added: "Pin 2 is left unconnected and will be a spare pin if needed"
- note added: "Room for a RC filter/voltage divider if needed"
- note added: "STOP is not used and the terminal block will be left depopulated unless we find a need for it."
- note added: "Three State LEDs all connect to the same GND pin"
Changed lines of the file:
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@@
 <text x="340.36" y="91.44" size="1.778" layer="91">Speaker</text>
 <text x="378.46" y="91.44" size="1.778" layer="91">TOF Sensor</text>
+<text x="22.86" y="93.98" size="1.778" layer="91">Female header pins for Arduino Nano.
+The microcontroller will get power from
+the 5V into the board</text>
+<text x="119.38" y="33.02" size="1.778" layer="91">STOP is not used and the terminal block
+will be left depopulated unless we find a
+need for it.</text>
+<text x="147.32" y="96.52" size="1.778" layer="91">Both servos use the same
+power terminal block</text>
+<text x="233.68" y="73.66" size="1.778" layer="91">Pin 2 is left unconnected and will
+be a spare pin if needed</text>
+<text x="266.7" y="60.96" size="1.778" layer="91">Three State LEDs all connect
+to the same GND pin</text>
+<text x="304.8" y="93.98" size="1.778" layer="91">Room for a RC filter/voltage
+divider if needed</text>
 </plain>
 <instances>
@@
 <attribute name="VALUE" x="317.5" y="68.58" size="1.778" layer="96"/>
 </instance>
+<instance part="IC1" gate="P" x="40.64" y="17.78" smashed="yes">
+<attribute name="NAME" x="40.005" y="17.145" size="1.778" layer="95"/>
+</instance>
 </instances>
 <busses>
@@
 <wire x1="222.25" y1="66.04" x2="223.52" y2="66.04" width="0.1524" layer="91"/>
 <pinref part="P+5" gate="1" pin="+5V"/>
+</segment>
+<segment>
+<pinref part="IC1" gate="P" pin="VCC"/>
+<wire x1="40.64" y1="25.4" x2="50.8" y2="25.4" width="0.1524" layer="91"/>
+<label x="48.26" y="25.4" size="1.778" layer="95"/>
 </segment>
 </net>
@@
 </drawing>
 <compatibility>
+<note version="6.3" minversion="6.2.2" severity="warning">
+Since Version 6.2.2 text objects can contain more than one line,
+which will not be processed correctly with this version.
+</note>
 <note version="8.2" severity="warning">
 Since Version 8.2, EAGLE supports online libraries. The ids
